File: electronics/radio.kicad_sch (KiCad schematic)
At the start: 33 parts, among them J7 SIM_Card, J9 Conn_Coaxial_Small, Q1 SI2302CDS, SW1 SW_Push, U2 TPS22953

Commit message: electronics: update dnp
Parts:
- SW1: now not fitted; now left out of the parts list
Changed lines of the file:
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@@
 		(body_style 1)
 		(exclude_from_sim no)
-		(in_bom yes)
+		(in_bom no)
 		(on_board yes)
-		(in_pos_files yes)
-		(dnp no)
+		(in_pos_files no)
+		(dnp yes)
 		(fields_autoplaced yes)
 		(property "Reference" "SW1"

Commit message: electronics: update MPNs and DNPs
Parts:
- C25, C26: MPN (none) -> TPSB107K006R0250
- R31: now left out of the parts list
Changed lines of the file:
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@@
+			)
+		)
+		(property "MPN" "TPSB107K006R0250"
+			(at 77.47 68.58 0)
+			(hide yes)
+			(show_name no)
+			(do_not_autoplace no)
+			(effects
+				(font
+					(size 1.27 1.27)
+				)
 			)
 		)
@@
 			)
 		)
+		(property "MPN" "TPSB107K006R0250"
+			(at 66.04 68.58 0)
+			(hide yes)
+			(show_name no)
+			(do_not_autoplace no)
+			(effects
+				(font
+					(size 1.27 1.27)
+				)
+			)
+		)
 		(pin "2"
 		)
@@
 		(body_style 1)
 		(exclude_from_sim no)
-		(in_bom yes)
-		(on_board yes)
-		(in_pos_files yes)
+		(in_bom no)
+		(on_board yes)
+		(in_pos_files no)
 		(dnp yes)
 		(fields_autoplaced yes)
