File: electronics/charger.kicad_sch (KiCad schematic)
At the start: 24 parts, among them J5 Conn_01x02_MountingPin, Q2 SI2302CDS, SW3 SW_SPDT, U6 TPS7A0518PDBV, U8 BQ25302RTER

Commit message: electronics: simplify BOM and fix issues
Parts:
- added J11: Conn_01x02_MountingPin, MyScale:JST_S2B-PH-SM4-TB(LF)(SN), symbol Connector_Generic_MountingPin:Conn_01x02_MountingPin
- added R32: 0R, Resistor_SMD:R_1206_3216Metric, symbol Device:R
- R10: value 390R -> 5.1k
- SW3: footprint MyScale:CAK_AYZ0102AURLC -> MyScale:NKK_CS12ANW03
Connections:
- net GND: now also J11.1 (Pin_1), J11.MP (MountPin)
- net REGN: now also D4.2 (A)
- net VBAT: now also R32.2
- net VBUS: no longer D4.2 (A)
- net Vpack: now also J11.2 (Pin_2), R32.1

Commit message: electronics: add values for charger
Parts:
- R32: now fitted; now in the parts list
- SW3: now not fitted; now left out of the parts list
Changed lines of the file:
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@@
 		(body_style 1)
 		(exclude_from_sim no)
-		(in_bom yes)
-		(on_board yes)
-		(in_pos_files yes)
-		(dnp no)
+		(in_bom no)
+		(on_board yes)
+		(in_pos_files no)
+		(dnp yes)
 		(fields_autoplaced yes)
 		(property "Reference" "SW3"
@@
 		(body_style 1)
 		(exclude_from_sim no)
-		(in_bom no)
-		(on_board yes)
-		(in_pos_files no)
-		(dnp yes)
+		(in_bom yes)
+		(on_board yes)
+		(in_pos_files yes)
+		(dnp no)
 		(fields_autoplaced yes)
 		(property "Reference" "R32"
