File: electronics/MyScale.kicad_sch (KiCad schematic)
At the start: 28 parts, among them J10 Conn_02x03_Odd_Even, J12 Conn_01x02_MountingPin, J8 Conn_01x02_MountingPin, U5 STM32U083CCUx, Y1 Crystal

Commit message: electronics: update dnp
Parts:
- J12: now not fitted; now left out of the parts list
Changed lines of the file:
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@@
 		(body_style 1)
 		(exclude_from_sim no)
-		(in_bom yes)
+		(in_bom no)
 		(on_board yes)
-		(in_pos_files yes)
-		(dnp no)
+		(in_pos_files no)
+		(dnp yes)
 		(property "Reference" "J12"
 			(at 69.85 -85.852 0)

Commit message: electronics: improve stencil openings for STM32
Parts:
- U5: footprint Package_DFN_QFN:QFN-48-1EP_7x7mm_P0.5mm_EP5.6x5.6mm -> MyScale:QFN-48-1EP_7x7mm_P0.5mm_EP5.6x5.6mm
Changed lines of the file:
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@@
 			)
 		)
-		(property "Footprint" "Package_DFN_QFN:QFN-48-1EP_7x7mm_P0.5mm_EP5.6x5.6mm"
+		(property "Footprint" "MyScale:QFN-48-1EP_7x7mm_P0.5mm_EP5.6x5.6mm"
 			(at 199.39 139.7 0)
 			(hide yes)

Commit message: electronics: update MPNs and DNPs
Parts:
- R5: now left out of the parts list
Changed lines of the file:
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@@
 		(body_style 1)
 		(exclude_from_sim no)
-		(in_bom yes)
+		(in_bom no)
 		(on_board yes)
-		(in_pos_files yes)
+		(in_pos_files no)
 		(dnp yes)
 		(property "Reference" "R5"
