File: electronics/BatteryAdapter/BatteryAdapter.kicad_sch (KiCad schematic)
At the start: 8 parts, among them J1 Conn_01x06_MountingPin, J2 Conn_01x02

Commit message: electronics: fix battery adapter pins
Parts:
- added R3, R4: 5.1k, Resistor_SMD:R_0603_1608Metric, symbol Device:R
Connections:
- net CC1: now also J1.5 (Pin_5); no longer J1.4 (Pin_4)
- net CC2: now also J1.4 (Pin_4); no longer J1.3 (Pin_3)
- net GND: now also R3.2, R4.2
- net D+: now reaches J1.2 (Pin_2)
- net D+: now also R3.1
- new net D-: J1.3 (Pin_3), R4.1

Commit message: batteryAdapter: prepare for pnp
Parts:
- J2: now left out of the parts list
Changed lines of the file:
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@@
 		(body_style 1)
 		(exclude_from_sim no)
-		(in_bom yes)
-		(on_board yes)
-		(in_pos_files yes)
+		(in_bom no)
+		(on_board yes)
+		(in_pos_files no)
 		(dnp no)
 		(fields_autoplaced yes)
@@
 		(in_bom no)
 		(on_board yes)
-		(in_pos_files yes)
+		(in_pos_files no)
 		(dnp no)
 		(fields_autoplaced yes)
@@
 		(in_bom no)
 		(on_board yes)
-		(in_pos_files yes)
+		(in_pos_files no)
 		(dnp no)
 		(fields_autoplaced yes)
@@
 		(in_bom no)
 		(on_board yes)
-		(in_pos_files yes)
+		(in_pos_files no)
 		(dnp no)
 		(fields_autoplaced yes)
@@
 		(in_bom no)
 		(on_board yes)
-		(in_pos_files yes)
-		(dnp no)
-		(fields_autoplaced yes)
+		(in_pos_files no)
+		(dnp no)
+		(fields_autoplaced yes)
